File: icatel.sch (KiCad schematic (older format))
At the start: 33 parts, among them CN6 CONN_13X2, CN7 CONN_8X2, CN8 CONN_13X2, X1 11.0592MHz

Commit message: Updating schematics based on further inspection of the pcb (using a multimeter).
Parts:
- added CI5: TLC254, symbol TLC254
- added D1, D10, D11, D29, D3, D36/NC, D4, D5, D6: DIODE, symbol DIODE
- added Q4: MPSA42, TO92-CBE, symbol MPSA42
- added Q?: MPSA92, TO92-CBE, symbol MPSA92
- added R19, R23, R24, R25, R46, R58, R59, R60, R91, R93, R95, R97: R, symbol R
Connections:
- net D0: now also CI12.3 (D0), CI16.3 (D0), CI8.3 (D0)
- net D1: now also CI12.4 (D1), CI16.4 (D1), CI8.4 (D1)
- net D2: now also CI12.7 (D2), CI16.7 (D2), CI8.7 (D2)
- net D3: now also CI12.8 (D3), CI16.8 (D3), CI8.8 (D3)
- net D4: now also CI12.13 (D4), CI16.13 (D4), CI8.13 (D4)
- net D5: now also CI12.14 (D5), CI16.14 (D5), CI8.14 (D5)
- net D6: now also CI12.17 (D6), CI16.17 (D6), CI8.17 (D6)
- net D7: now also CI12.18 (D7), CI16.18 (D7), CI8.18 (D7)
- net GND: now also D4.1 (A), D5.1 (A), Q4.E, R59.2
- net at CI8.12 (Q4): now also R91.2
- net at CI8.15 (Q5): now also R95.2
- net CN8_16: now reaches CI8.16 (Q6)
- net CN8_16: now also CN8.16 (P16)
- net at CI8.19 (Q7): now also R97.2
- net CI8_Q0: now reaches CI8.2 (Q0)
- net CI8_Q0: now also R60.1
- net at CI8.5 (Q1): now also R93.2
- net at CI8.6 (Q2): now also R46.2
- net at CI8.9 (Q3): now also D29.2 (K)
- net at CI12.15 (Q5): now also R25.2
- net at CI12.16 (Q6): now also D36/NC.2 (K)
- new net: Q4.B, R59.1, R60.2
- new net: Q4.C, R58.1
- new net: D10.1 (A), R19.1, R58.2
- new net: D10.2 (K), R19.2, R23.1
- new net: D3.2 (K), D6.2 (K), R23.2, R24.1
- new net: D1.2 (K), D3.1 (A), D4.2 (K)
- new net: D11.2 (K), D5.2 (K), D6.1 (A)
Other:
- note added: "(D13)"
- note added: "(Q13)"
- note added: "(Q2)"
- note added: "TriState Buffer"
- moved on the sheet: CI12, CI15, CI16, CI7A, CI7B, CI7C, CI7D, CI7F, CI8, D31, D32, D33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

Commit message: updating schematics
Parts:
- added CI20: X24C04, symbol X24C04
- added U?: TEA1063, symbol TEA1063
Connections:
- net +5V: now also CI20.8 (VCC)
- net DGND: now also CI20.1 (A0), CI20.2 (A1), CI20.3 (A2), CI20.4 (GND), CI20.7 (TEST)
- net EEPROM_SCL: now reaches CI13.13 (P3.3/~INT1)
- net EEPROM_SCL: now also CI20.6 (SCL)
- net EEPROM_SDA: now reaches CI13.8 (P1.7)
- net EEPROM_SDA: now also CI20.5 (SDA)
Other:
- note added: "Componentes que ainda não foram mapeados"
- note added: "I2C SERIAL EEPROM\n512kbytes"
- moved on the sheet: CI10A, CI10B, CI17, CI5A, CI5B, CI5C, CI5D, CI7A, CI7B, CI7C, CI7D, CI7E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
